File: kicad/pato/pato.kicad_pcb (KiCad board)
At the start: 2 copper layers, 99.1 x 40.6 mm, 21 parts, among them J1 DEBUG, J2 Conn_01x16, Q1 2N7002, Q2 AO3403A, U1 AMS1117-3.3, U2 ATtiny2313-20SU

Commit message: Add on-board pull-up option
Parts:
- added J3: SDA_PU, Pin_Headers:Pin_Header_Straight_1x02_Pitch2.54mm, F.Cu at (52.6, 92.0)
- added J4: SCK_PU, Pin_Headers:Pin_Header_Straight_1x02_Pitch2.54mm, F.Cu at (57.3, 92.0)
- added R4: 7.5K, Capacitors_SMD:C_0805_HandSoldering, F.Cu at (53.3, 87.6)
- added R5: 7.5K, Capacitors_SMD:C_0805_HandSoldering, F.Cu at (57.1, 87.6)
Routing:
- net /MOSI: track 18.1 -> 86.5 mm, vias 0 -> 2
- net +3V3: track 90.6 -> 149.7 mm, vias 2 -> 3
- net /SCK: track 47.4 -> 99.7 mm, vias 0 -> 2
- net Net-(J3-Pad1): track 0.00 -> 3.41 mm
- net Net-(J4-Pad1): track 0.00 -> 3.17 mm
- net +5VD: track 101.3 -> 102.7 mm
- net GND: track 48.9 -> 47.8 mm
Other:
- board text added: "Pato 20210531"
- board text removed: "Pato 20210522"
