File: kicad/aardwark/aardwark/aardwark.kicad_pcb (KiCad board)
At the start: 2 copper layers, 71.1 x 50.8 mm, 6 parts, among them J1 AARDWARK, J2 TEST, J3 PATO, J4 ICE, J5 POWER, J6 PW_JMP

Commit message: Add pinouts on F.Fab layer for Aardwark adapter
Other:
- board text added: "+5V"
- board text added: "+5VD"
- board text added: "GND"
- board text added: "MISO"
- board text added: "MOSI"
- board text added: "RESET"
- board text added: "SCK"
